File: ft230xs_usb2uart.kicad_pcb (KiCad board)
At the start: 2 copper layers, 40.9 x 20 mm, 21 parts, among them J1 USB_A, J2 Conn_01x04_Socket, SW1 SW_Push, U3 FT230XS

Commit message: adasd
Parts:
- moved SW1 34.9 mm to (136.4, 111.6)
- moved TX 30.1 mm to (151.5, 102.9), turned to 90 degrees
- moved C6 29.1 mm to (144.2, 111.2), turned to 90 degrees
- moved RX 27.4 mm to (149.6, 102.9), turned to 90 degrees
- moved R4 25.8 mm to (151.5, 107.1), turned to -90 degrees
- moved C8 25.0 mm to (140.3, 113.4), turned to -90 degrees
- moved R6 24.2 mm to (142.1, 111.8), turned to 90 degrees
- moved R5 22.8 mm to (149.6, 107.1), turned to -90 degrees
- moved U3 6.67 mm to (148.9, 114.5), turned to 180 degrees
- moved C2 6.07 mm to (135.7, 105.8)
- moved R1 6.07 mm to (138.9, 103.0)
- moved R2 6.07 mm to (138.9, 105.0)
- moved C3 5.19 mm to (134.8, 103.0), turned to 180 degrees
- moved C5 3.16 mm to (142.2, 115.5), turned to -90 degrees
- moved FB1 2.22 mm to (135.9, 115.6)
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- renumbered D1 to PWR, D3 to RX, D2 to TX
Connections:
- J2 pad 2: RXD -> TXD
- J2 pad 3: TXD -> RXD
- R6 pad 2: +3.3V -> +3V3
Routing:
- net +3V3: track 0.00 -> 28.7 mm, vias 0 -> 2
- net USB_D+: track 0.00 -> 26.5 mm
- net +5V: track 0.00 -> 26.2 mm
- net USB_D-: track 0.00 -> 23.6 mm
- net GND: track 0.00 -> 14.5 mm, vias 0 -> 10
- net RX_LED: track 0.00 -> 11.9 mm, vias 0 -> 2
- net TXD: track 0.00 -> 8.81 mm
- net TX_LED: track 0.00 -> 8.57 mm, vias 0 -> 2
- net ~{RST}: track 0.00 -> 8.55 mm
- net RXD: track 0.00 -> 8.52 mm
- net VBUS: track 0.00 -> 5.42 mm
- net /PWR_LED: track 0.00 -> 1.79 mm
Other:
- board text added: "KAJDEV Rev. 1.0"
- board text added: "USB2 UART"
- board text removed: "USB2UART"

Commit message: adasd
Routing:
- net GND: track 14.5 -> 15.6 mm
- net RX_LED: track 11.9 -> 12.9 mm
Other:
- board size 40.9 x 20 mm -> 41 x 20 mm
- board text added: "5V"
- board text added: "GND"
- board text added: "KAJDEV REV_1_0"
- board text added: "RXD"
- board text added: "TXD"
- board text removed: "KAJDEV Rev. 1.0"
Changed lines of the file:
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@@
 		(tags "resistor handsolder")
 		(property "Reference" "R4"
-			(at 0.01 -1.51 90)
+			(at 2.8175 0 180)
 			(layer "F.SilkS")
 			(effects
@@
 		)
 		(fp_line
-			(start 0.3 -2.1)
-			(end 0 -1.5)
-			(stroke
-				(width 0.12)
-				(type solid)
-			)
-			(layer "F.SilkS")
-		)
-		(fp_line
-			(start -0.3 -2.1)
-			(end 0.3 -2.1)
-			(stroke
-				(width 0.12)
-				(type solid)
-			)
-			(layer "F.SilkS")
-		)
-		(fp_line
-			(start 0 -1.5)
-			(end -0.3 -2.1)
-			(stroke
-				(width 0.12)
-				(type solid)
-			)
-			(layer "F.SilkS")
-		)
-		(fp_line
 			(start 8.64 2.09)
 			(end 3.75 2.09)
@@
 	)
 	(gr_rect
-		(start 163.3375 104.975)
-		(end 165.3375 114.975)
+		(start 159.82 104.975)
+		(end 161.82 114.975)
 		(stroke
 			(width 0.1)
@@
 		(layer "B.SilkS")
 	)
-	(gr_arc
-		(start 166.462578 116)
-		(mid 165.290982 118.828482)
-		(end 162.4625 120.000078)
-		(stroke
-			(width 0.05)
-			(type default)
-		)
-		(layer "Edge.Cuts")
-	)
-	(gr_arc
-		(start 162.4625 99.999922)
-		(mid 165.290982 101.171518)
-		(end 166.462578 104)
-		(stroke
-			(width 0.05)
-			(type default)
-		)
-		(layer "Edge.Cuts")
-	)
 	(gr_line
 		(start 125.5375 100)
@@
 	)
 	(gr_line
-		(start 166.462578 104)
-		(end 166.462578 116)
+		(start 166.54 100)
+		(end 166.54 120)
 		(stroke
 			(width 0.05)
@@
 	)
 	(gr_line
-		(start 162.4625 120.000124)
+		(start 166.54 120.000124)
 		(end 125.5375 120.000124)
 		(stroke
@@
 	(gr_line
 		(start 125.5375 100)
-		(end 162.4625 100)
+		(end 166.54 100)
 		(stroke
 			(width 0.05)
@@
 		(layer "Edge.Cuts")
 	)
-	(gr_text "KAJDEV\nRev. 1.0"
-		(at 160.05 115.13 270)
+	(gr_text "KAJDEV\nREV_1_0"
+		(at 162.35 115.13 270)
 		(layer "B.SilkS")
 		(effects
@@
 		)
 	)
+	(gr_text "5V"
+		(at 155.49 114.38 0)
+		(layer "F.SilkS")
+		(effects
+			(font
+				(size 1 1)
+				(thickness 0.15)
+			)
+			(justify right bottom)
+		)
+	)
+	(gr_text "RXD"
+		(at 155.49 109.38 0)
+		(layer "F.SilkS")
+		(effects
+			(font
+				(size 1 1)
+				(thickness 0.15)
+			)
+			(justify right bottom)
+		)
+	)
+	(gr_text "GND"
+		(at 155.49 106.88 0)
+		(layer "F.SilkS")
+		(effects
+			(font
+				(size 1 1)
+				(thickness 0.15)
+			)
+			(justify right bottom)
+		)
+	)
+	(gr_text "TXD"
+		(at 155.49 111.88 0)
+		(layer "F.SilkS")
+		(effects
+			(font
+				(size 1 1)
+				(thickness 0.15)
+			)
+			(justify right bottom)
+		)
+	)
 	(segment
 		(start 138.62 115.575)
@@
 	)
 	(segment
-		(start 153.18 110.86)
-		(end 153.18 103.7)
+		(start 153.18 110.09)
+		(end 153.18 103.695)
 		(width 0.5)
 		(layer "F.Cu")
@@
 	)
 	(segment
-		(start 153.18 103.7)
-		(end 153.1825 103.6975)
+		(start 153.18 103.695)
+		(end 151.52 102.035)
 		(width 0.5)
 		(layer "F.Cu")
@@
 	)
 	(segment
-		(start 153.1825 103.6975)
-		(end 151.52 102.035)
-		(width 0.5)
-		(layer "F.Cu")
-		(net 2)
-	)
-	(segment
 		(start 145.05 112.915)
 		(end 144.215 112.08)
@@
 	)
 	(via
-		(at 153.1825 114.7675)
+		(at 153.18 110.09)
 		(size 0.6)
 		(drill 0.3)
@@
 	)
 	(via
-		(at 153.18 110.86)
+		(at 153.1825 114.7675)
 		(size 0.6)
 		(drill 0.3)
@@
 	(segment
 		(start 153.1825 114.7675)
-		(end 153.1825 110.8625)
+		(end 153.1825 110.0925)
 		(width 0.5)
 		(layer "B.Cu")
@@
 	)
 	(segment
-		(start 153.1825 110.8625)
-		(end 153.18 110.86)
+		(start 153.1825 110.0925)
+		(end 153.18 110.09)
 		(width 0.5)
 		(layer "B.Cu")
@@
 	)
 	(segment
-		(start 146.285 114.82)
-		(end 145.65 114.82)
-		(width 0.5)
-		(layer "F.Cu")
-		(net 8)
-	)
-	(segment
 		(start 133.63 117.325)
 		(end 133.64 117.335)
@@
 	)
 	(segment
+		(start 147.32 114.82)
+		(end 147.34 114.84)
+		(width 0.5)
+		(layer "F.Cu")
+		(net 8)
+	)
+	(segment
 		(start 134.165 111.59)
 		(end 135.155 111.59)
@@
 	(segment
 		(start 146.285 114.82)
-		(end 146.3 114.805)
+		(end 147.32 114.82)
 		(width 0.5)
 		(layer "F.Cu")
@@
 	)
 	(segment
-		(start 145.65 114.82)
-		(end 144.095 116.375)
+		(start 133.65 117.325)
+		(end 133.64 117.335)
 		(width 0.5)
 		(layer "F.Cu")
@@
 	)
 	(segment
-		(start 133.65 117.325)
-		(end 133.64 117.335)
+		(start 144.095 116.375)
+		(end 145.65 114.82)
 		(width 0.5)
 		(layer "F.Cu")
@@
 		(net 8)
 	)
+	(segment
+		(start 145.65 114.82)
+		(end 146.285 114.82)
+		(width 0.5)
+		(layer "F.Cu")
+		(net 8)
+	)
 	(via
 		(at 150.48 113.98)
@@
 	)
 	(via
-		(at 133.64 117.335)
+		(at 147.34 114.84)
 		(size 0.6)
 		(drill 0.3)
@@
 	)
 	(via
-		(at 145.13 115.32)
+		(at 133.64 117.335)
 		(size 0.6)
 		(drill 0.3)
@@
 	)
 	(segment
-		(start 146.285 115.455)
-		(end 147.395 115.455)
+		(start 147.015 115.455)
+		(end 147.4 115.84)
 		(width 0.5)
 		(layer "F.Cu")
@@
 	)
 	(segment
-		(start 147.395 115.455)
-		(end 147.4 115.45)
+		(start 149.55 106.16)
+		(end 149.55 103.7725)
 		(width 0.5)
 		(layer "F.Cu")
@@
 	)
 	(segment
-		(start 149.55 106.16)
-		(end 149.55 103.7725)
+		(start 146.285 115.455)
+		(end 147.015 115.455)
 		(width 0.5)
 		(layer "F.Cu")
@@
 	)
 	(via
-		(at 147.4 115.45)
+		(at 147.4 115.84)
 		(size 0.6)
 		(drill 0.3)
@@
 	)
 	(segment
-		(start 147.4 115.45)
-		(end 147.4175 115.45)
+		(start 148.27 115.84)
+		(end 149.55 114.56)
 		(width 0.5)
 		(layer "B.Cu")
@@
 	)
 	(segment
-		(start 149.55 113.3)
-		(end 147.4 115.45)
+		(start 147.4 115.84)
+		(end 148.27 115.84)
 		(width 0.5)
 		(layer "B.Cu")
@@
 	)
 	(segment
-		(start 149.55 109.0125)
-		(end 149.55 113.3)
+		(start 149.55 114.56)
+		(end 149.55 109.0125)
 		(width 0.5)
 		(layer "B.Cu")
@@
 		(polygon
 			(pts
-				(xy 125.5375 100) (xy 166.4525 100) (xy 166.4525 120) (xy 125.5375 120)
+				(xy 125.5375 100) (xy 125.5375 120.000124) (xy 166.54 120.000124) (xy 166.54 100)
 			)
 		)
@@
 		(polygon
 			(pts
-				(xy 125.5375 100) (xy 166.4575 100) (xy 166.4575 120) (xy 125.5375 120)
+				(xy 125.5375 100) (xy 125.5375 120.000124) (xy 166.54 120.000124) (xy 166.54 100)
 			)
 		)
